File: projects/memi8M-01/memi8M-01.kicad_pcb (KiCad board)
At the start: 2 copper layers, 133.4 x 100.3 mm, 46 parts, among them J1 Conn_01x06, J2 Conn_01x02, J3 Conn_01x03, J4 Conn_01x06, SW1 SW_DIP_x05, U1 74HC595N, U10 74LS166N, U11 SST39VF1681_1682, U12 74LVC4245, U2 74HC595N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

Commit message: Prepared memi8M-01 for production. (Small fixes applied)
Routing:
- net GND_: track 1268.3 -> 1287.1 mm, vias 114 -> 127
